File: Electronics/LTDM_RevC/CurrentSense.kicad_sch (KiCad schematic)
At the start: 28 parts, among them SW2 SW_SP3T, U27 OPA1612AxD, U28 OPA1612AxD, U29 OPA2350

Commit message: Boards Ordered!
The KiCad files are the ones that were ordered
Parts:
- R2: LCSC C860931 -> C309660
Changed lines of the file:
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@@
 			)
 		)
-		(property "LCSC" "C860931"
+		(property "LCSC" "C309660"
 			(at 214.63 96.52 90)
 			(effects
