File: Electronics/LTDM_RevC/Preamp+Rectifier.kicad_sch (KiCad schematic)
At the start: 62 parts, among them J19 Conn_01x03_Male, J20 Conn_01x03_Male, J24 CSR_Bypass, J3 Conn_01x03_Male, J35 AudioJack3_SwitchTR, J37 AudioJack3_SwitchTR, J8 Conn_01x03_Male, U2 LF398_SOIC14, U22 OPA1612AxD, U24 OPA1612AxD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

Commit message: Boards Ordered!
The KiCad files are the ones that were ordered
Parts:
- J35, J37: LCSC (none) -> C4991610
- R103: LCSC C860931 -> C309660
- R11, R18: LCSC (none) -> C861645
Changed lines of the file:
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@@
+			)
+		)
+		(property "LCSC" "C861645"
+			(at 45.72 173.99 90)
+			(effects
+				(font
+					(size 1.27 1.27)
+				)
+				(hide yes)
 			)
 		)
@@
 		)
 		(property "Description" "Audio Jack, 3 Poles (Stereo / TRS), Switched TR Poles (Normalling)"
+			(at 373.38 83.82 0)
+			(effects
+				(font
+					(size 1.27 1.27)
+				)
+				(hide yes)
+			)
+		)
+		(property "LCSC" "C4991610"
 			(at 373.38 83.82 0)
 			(effects
@@
 			)
 		)
-		(property "LCSC" "C860931"
+		(property "LCSC" "C309660"
 			(at 342.9 184.15 90)
 			(effects
@@
 			)
 		)
+		(property "LCSC" "C861645"
+			(at 74.93 179.07 90)
+			(effects
+				(font
+					(size 1.27 1.27)
+				)
+				(hide yes)
+			)
+		)
 		(pin "1"
 		)
@@
 			(at 360.68 44.45 0)
 			(effects
+				(font
+					(size 1.27 1.27)
+				)
+				(hide yes)
+			)
+		)
+		(property "LCSC" "C4991610"
+			(at 360.68 44.45 0)
+			(effects
