File: Electronics/LTDM_RevC/LTDM_RevC.kicad_pcb (KiCad board)
At the start: 4 copper layers, 200 x 110 mm, 412 parts, among them J1 Conn_01x03_Male, J10 Conn_01x03_Male, J11 CSR_Bypass, J12 SpringTerminal, J13 Ban1, J14 CSR_Bypass, J15 SpringTerminal, J16 Barrel_Jack, J17 Ban2, J18 Conn_01x03_Male, J19 Conn_01x03_Male, J2 Conn_01x03_Male, J20 Conn_01x03_Male, J21 Conn_01x03_Male, J22 Barrel_Jack, J23 Conn_01x03_Male, J24 CSR_Bypass, J25 Ban3, J27 Conn_01x03_Male, J28 CSR_Bypass, J29 Conn_01x03_Male, J3 Conn_01x03_Male, J30 Conn_01x03_Male, J31 Conn_01x03_Male, J32 Conn_01x03_Male, J35 AudioJack3_SwitchTR, J36 AudioJack3_SwitchTR, J37 AudioJack3_SwitchTR, J38 AudioJack3_SwitchTR, J4 Conn_02x05_Odd_Even, J5 Conn_02x15_Odd_Even, J6 Conn_01x03_Male, J7 Conn_01x04_Socket, J8 Conn_01x03_Male, J9 Conn_01x03_Male, Q1 FQP27P06, Q15 BSS123, Q16 BSS123, Q2 IRLZ44N, Q3 FQP27P06, Q4 IRLZ44N, Q5 FQP27P06, Q6 IRLZ44N, SW1 SW_SP3T, SW2 SW_SP3T, SW3 SW_DPST, U1 74LVC1G11, U10 AP64500SP, U11 LM7332, U12 TC4427xOA, U13 OPA1612AxD, U14 OPA1612AxD, U15 LM393, U16 LF398_SOIC14, U17 OPA2350, U18 OPA1612AxD, U19 OPA1612AxD, U2 LF398_SOIC14, U20 74AUC2G86, U21 OPA2350, U22 OPA1612AxD, U23 OPA1612AxD, U24 OPA1612AxD, U25 OPA1612AxD, U26 74LVC1G11, U27 OPA1612AxD, U28 OPA1612AxD, U29 OPA2350, U3 OPA2350, U30 OPA1612AxD, U31 74LVC1G11, U32 74LVC1G11, U36 74LVC2G74, U4 OPA1612AxD, U5 LM393, U6 OPA1612AxD, U7 Teensy4.1A, U8 Teensy4.1B, U9 TC4426

Commit message: Synchronize TMC2209 motor drivers with LTDM
the ALT_SENSE pin now outputs a ~12.5MHz pulse wave that connects to BIGTREETECH TMC2209 Motor driver clock (CLK) inputs. This synchronizes the motor actuation events with the LTDM actuation events to avoid aliasing and crosstalk.
Parts:
- added C21: C_Small_US, Capacitor_THT:C_Rect_L11.0mm_W4.3mm_P10.00mm_MKT, F.Cu at (324.7, 118.2)
- added C47: C_Small_US, Capacitor_THT:C_Rect_L11.0mm_W4.3mm_P10.00mm_MKT, F.Cu at (345.5, 118.3)
- C4: moved to B.Cu
- moved C4 2.54 mm to (232.2, 91.3)
Routing:
- net MagIn2: track 129.7 -> 143.3 mm, vias 8 -> 10
