File: Electronics/LTDM_UI_RevC/LTDM_UI_RevC.kicad_pcb (KiCad board)
At the start: 2 copper layers, 200 x 110 mm, 76 parts, among them J21 NMJ6HCD2, J22 NMJ6HCD2, J24 Conn_02x15_Odd_Even, SW1 tactile, SW10 SW_Push_DPDT, SW11 SW_Push_DPDT, SW12 SW_Push_DPDT, SW13 SW_Push_DPDT, SW14 SW_Push_DPDT, SW15 SW_Push_DPDT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

Commit message: Boards Ordered!
The KiCad files are the ones that were ordered
Parts:
- removed SL1, SL2, SL3, SL4, SL5, SL6, SL7, SL8: 10k, Potentiometer_THT:Potentiometer_Bourns_PTA4543_Single_Slide
- added G***: LOGO, LOGO, F.Cu at (224.7, 56.3)
- added G***: LOGO, LOGO, B.Cu at (110.4, 143.2)
- added G***: LOGO, LOGO, B.Cu at (113.1, 62.5)
- added H5: MountingHole_Pad, MountingHole:MountingHole_4.3mm_M4_ISO14580_Pad, F.Cu at (148.8, 51.3)
- added J4: Conn_02x15_Odd_Even, Connector_IDC:IDC-Header_2x15_P2.54mm_Vertical_SILKSCREEN, B.Cu at (224.2, 105.1)
- added R3: 100, Resistor_SMD:R_0603_1608Metric, F.Cu at (202.8, 59.6)
- added R4: 100, Resistor_SMD:R_0603_1608Metric, F.Cu at (176.9, 59.6)
- added VR1: RS45111A900F, RS45111A900F:RS45111A900F, F.Cu at (155.0, 80.7)
- added VR2: RS45111A900F, RS45111A900F:RS45111A900F, F.Cu at (168.4, 80.7)
- added VR3: RS45111A900F, RS45111A900F:RS45111A900F, F.Cu at (181.7, 80.7)
- added VR4: RS45111A900F, RS45111A900F:RS45111A900F, F.Cu at (195.1, 80.7)
- added VR5: RS45111A900F, RS45111A900F:RS45111A900F, F.Cu at (208.5, 80.7)
- added VR6: RS45111A900F, RS45111A900F:RS45111A900F, F.Cu at (221.9, 80.7)
- added VR7: RS45111A900F, RS45111A900F:RS45111A900F, F.Cu at (235.3, 80.8)
- added VR8: RS45111A900F, RS45111A900F:RS45111A900F, F.Cu at (248.7, 80.8)
- moved R27 81.5 mm to (98.5, 138.0)
- moved R26 81.5 mm to (88.4, 138.0)
- moved R28 81.5 mm to (108.5, 138.1)
- moved R32 81.5 mm to (148.7, 138.8)
- moved R25 81.4 mm to (79.3, 138.0)
- moved R30 81.1 mm to (128.5, 138.1)
- moved R29 81.1 mm to (118.5, 138.1)
- moved R31 81.1 mm to (138.5, 138.3)
- moved SW1 80.1 mm to (74.3, 62.7), turned to -90 degrees
- moved SW10 80.1 mm to (84.2, 142.9)
- moved SW11 80.1 mm to (94.2, 142.9)
- moved SW12 80.1 mm to (104.2, 142.9)
- moved SW13 80.1 mm to (114.2, 142.9)
- moved SW14 80.1 mm to (124.2, 142.9)
- moved SW15 80.1 mm to (134.2, 142.9)
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Connections:
- J21 pad R: +3.3V -> Net-(J21-PadR)
- J21 pad RN: +3.3V -> unconnected-(J21-PadRN)
- J21 pad SN: GND -> unconnected-(J21-PadSN)
- J21 pad TN: FP1 -> unconnected-(J21-PadTN)
- J22 pad R: +3.3V -> Net-(J22-PadR)
- J22 pad RN: +3.3V -> unconnected-(J22-PadRN)
- J22 pad SN: GND -> unconnected-(J22-PadSN)
- J22 pad TN: FP2 -> unconnected-(J22-PadTN)
Routing:
- net +3.3V: track 798.9 -> 899.1 mm, vias 14 -> 11
- net SW8: track 100.0 -> 22.5 mm
- net SW7: track 109.6 -> 33.8 mm
- net SW1: track 167.2 -> 91.5 mm
- net SW6: track 119.2 -> 45.0 mm
- net SW5: track 128.8 -> 56.0 mm
- net SW4: track 138.4 -> 67.0 mm
- net SW3: track 148.0 -> 78.4 mm
- net SW2: track 157.6 -> 89.6 mm
- net BT8: track 23.6 -> 88.3 mm
- net BT7: track 34.3 -> 92.4 mm
- net BT6: track 45.3 -> 101.8 mm
- net BT5: track 56.3 -> 111.4 mm
- net BT4: track 67.7 -> 121.0 mm
- net BT3: track 78.6 -> 130.7 mm
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Other:
- board text added: "A.Read"
- board text added: "AS0"
- board text added: "AS1"
- board text added: "AS2"
- board text added: "AS3"
- board text added: "DS0"
- board text added: "DS1"
- board text added: "DS2"
- board text added: "DS3"
- board text added: "Dig.Read"
- board text added: "FP1"
- board text added: "FP2"
- board text added: "GND"
- board text added: "LEDs moved up by 2mm"
- board text added: "MOSI"
- board text added: "SCK"
- board text added: "~{LAT}"
- board text removed: "Lorentz TDM Board O' Knobs RevA 9/2025"
