File: Electronics/LTDM_UI_RevC/LTDM_UI_RevC.kicad_sch (KiCad schematic)
At the start: 79 parts, among them J19 Conn_01x04, J21 NMJ6HCD2, J22 NMJ6HCD2, J23 Conn_01x04, J24 Conn_02x15_Odd_Even, SW1 tactile, SW10 SW_Push_DPDT, SW11 SW_Push_DPDT, SW12 SW_Push_DPDT, SW13 SW_Push_DPDT, SW14 SW_Push_DPDT, SW15 SW_Push_DPDT, SW16 SW_Push_DPDT, SW2 tactile, SW3 tactile, SW4 tactile, SW5 tactile, SW6 tactile, SW7 tactile, SW8 tactile, SW9 SW_Push_DPDT, U1 TLC5947RHB, U18 74AHCT125, U2 CD74HC4067SM, U3 CD74HC4067SM

Commit message: Boards Ordered!
The KiCad files are the ones that were ordered
Parts:
- removed J19, J23: Conn_01x04, symbol Connector_Generic:Conn_01x04
- removed SL1, SL2, SL3, SL4, SL5, SL6, SL7, SL8: 10k, Potentiometer_THT:Potentiometer_Bourns_PTA4543_Single_Slide, symbol Device:R_Potentiometer_US
- removed U18: 74AHCT125, symbol 74xx:74AHCT125
- added H5: MountingHole_Pad, MountingHole:MountingHole_4.3mm_M4_ISO14580_Pad, symbol Mechanical:MountingHole_Pad
- added J1, J2, J3: Conn_01x03_Male, symbol Connector:Conn_01x03_Male
- added J4: Graphic, Connector_IDC:IDC-Header_2x15_P2.54mm_Vertical_SILKSCREEN, symbol Connector_Generic:Conn_02x15_Odd_Even
- added R3, R4: 100, Resistor_SMD:R_0603_1608Metric, symbol 1A_Favorites:R_Standard_Thru
- added VR1, VR2, VR3, VR4, VR5, VR6, VR7, VR8: RS45111A900F, RS45111A900F:RS45111A900F, symbol RS45111A900F:RS45111A900F
Connections:
- net +3.3V: now also R3.1, R4.1, VR1.1 (CCW), VR2.1 (CCW), VR3.1 (CCW), VR4.1 (CCW), VR5.1 (CCW), VR6.1 (CCW), VR7.1 (CCW), VR8.1 (CCW); no longer J21.R, J21.RN, J22.R, J22.RN
- net FP1: no longer J21.TN
- net FP2: no longer J22.TN
- net GND: now also H5.1, VR1.3 (CW), VR1.4 (MH1), VR1.5 (MH2), VR2.3 (CW), VR2.4 (MH1), VR2.5 (MH2), VR3.3 (CW), VR3.4 (MH1), VR3.5 (MH2), VR4.3 (CW), VR4.4 (MH1), VR4.5 (MH2), VR5.3 (CW), VR5.4 (MH1), VR5.5 (MH2), VR6.3 (CW), VR6.4 (MH1), VR6.5 (MH2), VR7.3 (CW), VR7.4 (MH1), VR7.5 (MH2), VR8.3 (CW), VR8.4 (MH1), VR8.5 (MH2); no longer J21.SN, J22.SN
- net SL1: now also VR1.2 (WIPER)
- net SL2: now also VR2.2 (WIPER)
- net SL3: now also VR3.2 (WIPER)
- net SL4: now also VR4.2 (WIPER)
- net SL5: now also VR5.2 (WIPER)
- net SL6: now also VR6.2 (WIPER)
- net SL7: now also VR7.2 (WIPER)
- net SL8: now also VR8.2 (WIPER)
- new net: J21.R, R4.2
- new net: J22.R, R3.2
- new net SH_in: J1.1 (Pin_1), J3.3 (Pin_3)
- new net rect_in: J2.3 (Pin_3), J3.1 (Pin_1)
- new net return: J2.2 (Pin_2)
- new net stage1out: J1.2 (Pin_2)
- new net stage2in: J1.3 (Pin_3), J2.1 (Pin_1)
- new net stage2out: J3.2 (Pin_2)
Other:
- note added: "(Changed from bourns PTA4543 to RS45111A900F due to availability on JLCPCB)"
- note added: "Ch1: J19 - Ch2: J27"
- note added: "Ch1: J20 - Ch2: J30"
- note added: "Ch1: J3 - Ch2: J21"
- note added: "Mode 1: S&H is pre-gain2 gain 1 -> S&H -> gain 2 [x][x][ ] [x][x][ ] [x][x][ ] Mode 2: S&H is post gain2 gain 1 -> gain 2 -> S&H [ ][x][x] [ ][x][x] [ ][x][x] Mode 3: bypass S&H gain 1 -> gain 2 [ ][x][x] [ ][ ][ ] [x][x][ ]"
- note added: "Mode 4: Teensy does not see S&H but SEND does [x][x][x] [ ][ ][ ] [x][x][ ] Mode 5: External audio input with gain [ ][ ][ ] <- doesn't matter really [x][x][ ] [x][x][ ] Mode 5: External audio input without gain [ ][ ][ ] <- doesn't matter really [ ][x][x] [ ][ ][ ] <- doesn't matter really"
- note added: "Routing Options"
- note added: "This is a graphic on the back of the PCB for helping use the main PCB"
- note removed: "should it be teensy 5V instead?"
- moved on the sheet: C5, CU1, CU10, CU11, CU12, CU2, CU3, CU5, CU6, CU7, CU8, CU9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
